File: hardware/QT1.kicad_pcb (KiCad board)
At the start: 2 copper layers, 40 x 55 mm, 12 parts, among them U1 TLE2141CD, U2 AD8561ARZ, U3 MCP601-xOT, U4 Teensy 4.0

Commit message: Add files via upload
Parts:
- added C3: 75pF, Capacitor_SMD:C_0603_1608Metric, F.Cu at (124.5, 117.0)
- U3: value MCP601-xOT -> MCP601-xSN; footprint Package_TO_SOT_SMD:SOT-23-5 -> Package_SO:SOIC-8_3.9x4.9mm_P1.27mm
- moved R3 1.19 mm to (124.5, 106.0)
- moved U4 0.83 mm to (140.0, 92.7)
- moved C2 0.76 mm to (124.5, 114.2)
- moved R4 0.76 mm to (124.6, 109.5)
- moved R5 0.76 mm to (128.8, 109.5)
- moved C1 0.52 mm to (128.8, 114.2)
- moved U3 0.51 mm to (154.5, 85.5)
Connections:
- C2 pad 2: GND1 -> Net-(C2-Pad2)
- U3 pad 1: Net-(U2-+) -> unconnected-(U3-NC-Pad1)
- U3 pad 2: GND3 -> Net-(U3--)
- U3 pad 4: Net-(U3--) -> GND3
- U3 pad 5: +5V -> unconnected-(U3-NC-Pad5)
Routing:
- net Net-(U2-+): track 46.0 -> 61.5 mm
- net Net-(D1-A): track 16.5 -> 26.5 mm
- net GND1: track 59.1 -> 66.9 mm, vias 0 -> 1
- net Net-(U3--): track 12.9 -> 20.2 mm
- net +5V: track 53.9 -> 47.4 mm, vias 0 -> 1
- net Net-(C2-Pad2): track 0.00 -> 2.84 mm
- net GND3: track 14.0 -> 16.1 mm
- net Net-(U2-~{Q}): track 20.7 -> 19.3 mm
- net Net-(R5-Pad1): track 11.0 -> 11.6 mm
- net Net-(D1-K): track 15.3 -> 15.7 mm, vias 1 -> 0
